File: DJI_A/_autosave-DJI_A.sch (KiCad schematic (older format))
At the start: 3 parts, among them J1 Conn_01x26, J2 Conn_01x26, J3 Conn_02x13_Odd_Even

Commit message: Unrouted DJI_A PCB added
Parts:
- J1, J2: footprint (none) -> UserLib:DF56C-26S
- J3: footprint (none) -> Connector_PinHeader_2.54mm:PinHeader_2x13_P2.54mm_Vertical
Changed lines of the file:
@@
 F 0 "J2" H 4200 3350 50  0000 C CNN
 F 1 "Conn_01x26" H 4200 650 50  0000 C CNN
-F 2 "" H 4200 2050 50  0001 C CNN
+F 2 "UserLib:DF56C-26S" H 4200 2050 50  0001 C CNN
 F 3 "~" H 4200 2050 50  0001 C CNN
 	1    4200 2050
@@
 F 0 "J1" H 1100 3450 50  0000 C CNN
 F 1 "Conn_01x26" H 1100 750 50  0000 C CNN
-F 2 "" H 1100 2150 50  0001 C CNN
+F 2 "UserLib:DF56C-26S" H 1100 2150 50  0001 C CNN
 F 3 "~" H 1100 2150 50  0001 C CNN
 	1    1100 2150
@@
 F 0 "J3" H 2700 4950 50  0000 C CNN
 F 1 "Conn_02x13_Odd_Even" H 2700 3550 50  0000 C CNN
-F 2 "" H 2650 4250 50  0001 C CNN
+F 2 "Connector_PinHeader_2.54mm:PinHeader_2x13_P2.54mm_Vertical" H 2650 4250 50  0001 C CNN
 F 3 "~" H 2650 4250 50  0001 C CNN
 	1    2650 4250
